File: wacky-waver.kicad_sch (KiCad schematic)
At the start: 0 parts

Commit message: feat(schematic): design MVP
Parts:
- added C1: C_US, symbol Device:C_US
- added J1: Conn_01x02_Pin, symbol Connector:Conn_01x02_Pin
- added Q1: RD3P050SNTL1 or FQD13N10LTM, Package_TO_SOT_SMD:TO-252-2, symbol Transistor_FET:SUD50P10-43L
- added U1: XIAO-ESP32-C5-SMD, Seeed_Studio_XIAO_Series:XIAO-ESP32-C5-SMD, symbol Seeed Xiao:XIAO-ESP32-C5-SMD
Connections:
- new net: J1.1 (Pin_1), Q1.2 (D)
- new net GNDPWR: C1.2, Q1.3 (S), U1.13 (GND), U1.27 (GND), U1.33 (GND)
- new net Motor Control: Q1.1 (G), U1.1 (GPIO1_A0_D0)
- new net VCC: C1.1, J1.2 (Pin_2), U1.14 (VBUS)
- no-connect marks 0 -> 20
Other:
- note added: "Use FQD for bang/bang. Use RD3 for analog control."
- title: (none) -> Wacky Waver

Commit message: feat(pcb): place initial components
Parts:
- C1: footprint (none) -> Capacitor_THT:C_Radial_D10.0mm_H20.0mm_P5.00mm
- J1: footprint (none) -> Connector_JST:JST_PH_B2B-PH-K_1x02_P2.00mm_Vertical
- U1: footprint Seeed_Studio_XIAO_Series:XIAO-ESP32-C5-SMD -> SEEED Xiao:XIAO-ESP32-C5-SMD
Changed lines of the file:
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@@
 			)
 		)
-		(property "Footprint" ""
+		(property "Footprint" "Capacitor_THT:C_Radial_D10.0mm_H20.0mm_P5.00mm"
 			(at 38.1 100.33 0)
 			(hide yes)
@@
 		(dnp no)
 		(fields_autoplaced yes)
-		(property "Reference" "#PWR04"
+		(property "Reference" "#PWR02"
 			(at 74.93 113.03 0)
 			(hide yes)
@@
 			(project "wacky-waver"
 				(path "/0fb331f2-2851-4e78-9031-6723af8f3488"
-					(reference "#PWR04")
+					(reference "#PWR02")
 					(unit 1)
 				)
@@
 		(dnp no)
 		(fields_autoplaced yes)
-		(property "Reference" "#PWR01"
+		(property "Reference" "#PWR04"
 			(at 198.12 68.58 0)
 			(hide yes)
@@
 			(project "wacky-waver"
 				(path "/0fb331f2-2851-4e78-9031-6723af8f3488"
-					(reference "#PWR01")
+					(reference "#PWR04")
 					(unit 1)
 				)
@@
 			)
 		)
-		(property "Footprint" ""
+		(property "Footprint" "Connector_JST:JST_PH_B2B-PH-K_1x02_P2.00mm_Vertical"
 			(at 80.01 91.44 0)
 			(hide yes)
@@
 		(dnp no)
 		(fields_autoplaced yes)
-		(property "Reference" "#PWR02"
+		(property "Reference" "#PWR05"
 			(at 198.12 132.08 0)
 			(hide yes)
@@
 			(project "wacky-waver"
 				(path "/0fb331f2-2851-4e78-9031-6723af8f3488"
-					(reference "#PWR02")
+					(reference "#PWR05")
 					(unit 1)
 				)
@@
 		(dnp no)
 		(fields_autoplaced yes)
-		(property "Reference" "#PWR05"
+		(property "Reference" "#PWR01"
 			(at 74.93 90.17 0)
 			(hide yes)
@@
 			(project "wacky-waver"
 				(path "/0fb331f2-2851-4e78-9031-6723af8f3488"
-					(reference "#PWR05")
+					(reference "#PWR01")
 					(unit 1)
 				)
@@
 			)
 		)
-		(property "Footprint" "Seeed_Studio_XIAO_Series:XIAO-ESP32-C5-SMD"
+		(property "Footprint" "SEEED Xiao:XIAO-ESP32-C5-SMD"
 			(at 157.48 91.44 0)
 			(hide yes)
